File: kicad/mss-atlasadapter.kicad_pcb (KiCad board)
At the start: 2 copper layers, 73.7 x 38.1 mm, 36 parts, among them J1 Screw_Terminal_01x02, J2 AVR-ISP, J3 8P8C, J4 8P8C, SW1 FSM4JSMATR, T1 PE-51687, U1 AP7381-33Y, U2 INA180A4, U3 ATtiny85-20S, U4 TLP241A

Commit message: First cut at board layout for the adapter
Parts:
- removed F1: 1210L020WR, Resistor_SMD:R_1210_3225Metric
- removed SW1: FSM4JSMATR, ISE_Generic:TE_FSM4JSMA
- removed T1: PE-51687, ISE_Generic:XFMR_PE-51687
- added C11: 10uF, Capacitor_SMD:C_0805_2012Metric, F.Cu at (56.3, 185.7)
- added C13: 0.1uF, Capacitor_SMD:C_0805_2012Metric, F.Cu at (72.1, 154.8)
- added C7: 0.1uF, Capacitor_SMD:C_0805_2012Metric, F.Cu at (43.6, 155.3)
- added C8: 0.1uF, Capacitor_SMD:C_0805_2012Metric, F.Cu at (37.3, 155.3)
- added D10: CDBM140G, ISE_Generic:SOD-123T, F.Cu at (58.4, 179.5)
- added D11: BLUE, LED_SMD:LED_0805_2012Metric, F.Cu at (82.9, 165.9)
- added L1: 4.7uH, ISE_UltraLibrarian:MSS6132-xxxMLC, F.Cu at (52.7, 179.5)
- added Q1: ZXMS6004FF, Package_TO_SOT_SMD:SOT-23, F.Cu at (58.7, 169.0)
- added Q2: ZXMS6004FF, Package_TO_SOT_SMD:SOT-23, F.Cu at (58.7, 173.2)
- added Q3: ZXMS6004FF, Package_TO_SOT_SMD:SOT-23, F.Cu at (58.7, 164.8)
- added R10: 10k, Resistor_SMD:R_0805_2012Metric, F.Cu at (70.2, 170.2)
- added R11: 10k, Resistor_SMD:R_0805_2012Metric, F.Cu at (63.1, 174.9)
- added R12: 10k, Resistor_SMD:R_0805_2012Metric, F.Cu at (77.5, 170.2)
- added R13: 10k, Resistor_SMD:R_0805_2012Metric, F.Cu at (63.1, 177.8)
- added R14: 1k, Resistor_SMD:R_0805_2012Metric, F.Cu at (77.2, 144.8)
- added R15: 10k, Resistor_SMD:R_0805_2012Metric, F.Cu at (59.3, 185.7)
- added R16: 10k, Resistor_SMD:R_0805_2012Metric, F.Cu at (63.1, 186.6)
- added R17: 1k, Resistor_SMD:R_0805_2012Metric, F.Cu at (66.7, 185.8)
- added R18: 1k, Resistor_SMD:R_0805_2012Metric, F.Cu at (63.1, 183.7)
- added R19: 330, Resistor_SMD:R_0805_2012Metric, F.Cu at (63.1, 180.7)
- added R20: 1k, Resistor_SMD:R_0805_2012Metric, F.Cu at (77.2, 147.7)
- added R21: 1k, Resistor_SMD:R_0805_2012Metric, F.Cu at (77.5, 157.6)
- added R22: 1k, Resistor_SMD:R_0805_2012Metric, F.Cu at (77.5, 160.5)
- added R23: 1k, Resistor_SMD:R_0805_2012Metric, F.Cu at (77.5, 163.4)
- added R7: 10k, Resistor_SMD:R_0805_2012Metric, F.Cu at (50.0, 152.4)
- added R8: 10k, Resistor_SMD:R_0805_2012Metric, F.Cu at (37.3, 149.6)
- added R9: 10k, Resistor_SMD:R_0805_2012Metric, F.Cu at (37.3, 152.4)
- added TP1: TestPoint, TestPoint:TestPoint_Pad_D2.0mm, B.Cu at (28.3, 175.3)
- added TP2: TestPoint, TestPoint:TestPoint_Pad_D2.0mm, B.Cu at (28.3, 180.3)
- C3: value 1uF -> 0.1uF
- D1, D2, D3, D4: footprint Diode_SMD:D_SOD-123 -> ISE_Generic:SOD-123T
- D5: value BAV99 -> BLUE; footprint Package_TO_SOT_SMD:SOT-23 -> LED_SMD:LED_0805_2012Metric
- D6: value GREEN LED -> AMBER
- D7: value RED LED -> RED
- D8: value AMBER LED -> AMBER
- D9: value SMAJ18A-TP -> GREEN LED; footprint Diode_SMD:D_SMA -> LED_SMD:LED_0805_2012Metric
- J1: value Screw_Terminal_01x02 -> 6P6C; footprint TerminalBlock_RND:TerminalBlock_RND_205-00012_1x02_P5.00mm_Horizontal -> Connector_RJ:RJ12_Amphenol_54601
- J2: value AVR-ISP -> 6P6C; footprint Connector:Tag-Connect_TC2030-IDC-NL_2x03_P1.27mm_Vertical -> Connector_RJ:RJ12_Amphenol_54601
- J3: value 8P8C -> Screw_Terminal_01x02; footprint Connector_RJ:RJ45_Amphenol_54602-x08_Horizontal -> TerminalBlock_RND:TerminalBlock_RND_205-00012_1x02_P5.00mm_Horizontal
- R2: value 1k -> 10k
- R3: value 1k -> 330
- R4: value 510 -> 330
- R5: value 100k -> 10k
- R6: value 330 -> 10k
- U1: value AP7381-33Y -> AP7381-50Y
- U2: value INA180A4 -> AP3012
- U3: value ATtiny85-20S -> 74HC4049; footprint Package_SO:SOIC-8W_5.3x5.3mm_P1.27mm -> Package_SO:SO-16_3.9x9.9mm_P1.27mm
- U4: value TLP241A -> 74HC4049; footprint ISE_UltraLibrarian:11-5B201S_TOS -> Package_SO:SO-16_3.9x9.9mm_P1.27mm
- moved D6 51.3 mm to (82.9, 146.8), turned to -90 degrees
- moved D5 46.4 mm to (82.9, 140.5)
- moved J3 45.5 mm to (32.3, 175.3), turned to -90 degrees
- moved D9 39.5 mm to (34.5, 160.9), turned to 90 degrees
- moved R2 39.1 mm to (50.0, 149.6), turned to 180 degrees
- moved D7 38.1 mm to (82.9, 153.2), turned to -90 degrees
- moved D8 37.0 mm to (82.9, 159.5), turned to -90 degrees
- moved R6 36.9 mm to (43.6, 152.4)
- moved R3 36.2 mm to (66.0, 149.6), turned to 180 degrees
- moved J2 35.3 mm to (67.7, 145.7), turned to 180 degrees
- moved J1 32.0 mm to (44.7, 145.7), turned to 180 degrees
- moved R1 28.1 mm to (37.5, 160.9), turned to -90 degrees
- moved H2 28.0 mm to (122.7, 185.4)
- moved R5 27.3 mm to (43.6, 149.6)
- moved H3 25.7 mm to (90.9, 132.6)
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Connections:
- C2 pad 1: +3.3V -> +5V
- C3 pad 1: /DCC_CURRENT -> Net-(C3-Pad1)
- C4 pad 1: /~{CAL_SW} -> Net-(C4-Pad1)
- C5 pad 1: +3.3V -> +5V
- C6 pad 2: +3.3V -> GND
- D5 pad 1: Net-(C6-Pad1) -> GND
- D5 pad 2: Net-(C6-Pad1) -> Net-(D5-Pad2)
- D9 pad 1: /MSS_OCC -> GND
- D9 pad 2: /MSS_GND -> Net-(D9-Pad2)
- J1 pad 1: Net-(D1-Pad2) -> unconnected-(J1-Pad1)
- J1 pad 2: Net-(D2-Pad2) -> Net-(J1-Pad2)
- J2 pad 1: Net-(J2-Pad1) -> unconnected-(J2-Pad1)
- J2 pad 2: +3.3V -> Net-(J1-Pad2)
- J2 pad 4: Net-(J2-Pad4) -> unconnected-(J2-Pad4)
- J2 pad 6: GND -> unconnected-(J2-Pad6)
- J3 pad 1: Net-(J3-Pad1) -> Net-(D1-Pad2)
- J3 pad 2: Net-(J3-Pad2) -> Net-(D2-Pad2)
- J4 pad 1: Net-(J3-Pad3) -> Net-(J4-Pad1)
- J4 pad 2: Net-(J3-Pad6) -> Net-(J4-Pad2)
- J4 pad 3: Net-(J3-Pad1) -> Net-(J4-Pad3)
- J4 pad 4: /MSS_OCC -> Net-(J4-Pad4)
- J4 pad 5: /MSS_GND -> GND
- J4 pad 6: Net-(J3-Pad2) -> Net-(J4-Pad6)
- J4 pad 7: Net-(J3-Pad7) -> unconnected-(J4-Pad7)
- J4 pad 8: Net-(J3-Pad8) -> unconnected-(J4-Pad8)
- R1 pad 1: Net-(D6-Pad2) -> Net-(D9-Pad2)
- R1 pad 2: +3.3V -> +5V
- R2 pad 1: Net-(J2-Pad1) -> +5V
- R2 pad 2: Net-(D7-Pad2) -> Net-(J1-Pad2)
- R3 pad 1: Net-(J2-Pad4) -> Net-(R3-Pad1)
- R3 pad 2: Net-(D8-Pad2) -> Net-(J2-Pad3)
- R4 pad 1: +3.3V -> Net-(R4-Pad1)
- R4 pad 2: Net-(C6-Pad1) -> Net-(J2-Pad5)
- R5 pad 1: /DCC_CURRENT -> +5V
- R5 pad 2: Net-(R5-Pad2) -> Net-(J1-Pad3)
- R6 pad 1: Net-(R6-Pad1) -> Net-(C7-Pad1)
- R6 pad 2: Net-(J2-Pad1) -> Net-(J1-Pad3)
- U1 pad 1: +3.3V -> +5V
- U2 pad 1: Net-(R5-Pad2) -> Net-(D10-Pad2)
- U2 pad 3: Net-(C6-Pad1) -> Net-(R16-Pad1)
- U2 pad 4: +3.3V -> +5V
- U2 pad 5: +3.3V -> +5V
- U3 pad 1: Net-(J2-Pad5) -> +5V
- U3 pad 2: /~{CAL_SW} -> Net-(R3-Pad1)
- U3 pad 3: /DCC_CURRENT -> /A_MSS_OUT
- U3 pad 4: GND -> /A_MSS_OUT
- U3 pad 5: Net-(J2-Pad4) -> Net-(C3-Pad1)
- U3 pad 6: Net-(J2-Pad1) -> Net-(R4-Pad1)
- U3 pad 7: Net-(J2-Pad3) -> /AA_MSS_OUT
- U3 pad 8: +3.3V -> GND
- U4 pad 1: Net-(R6-Pad1) -> +5V
- U4 pad 2: GND -> /S_MSS_IN
- U4 pad 3: /MSS_GND -> Net-(C6-Pad1)
- U4 pad 4: Net-(F1-Pad2) -> /A_MSS_IN
Routing:
- net +5V: track 0.00 -> 119.3 mm, vias 0 -> 10
- net +3.3V: track 61.5 -> 0.00 mm
- net /AA_MSS_IN: track 0.00 -> 44.8 mm, vias 0 -> 2
- net /AA_MSS_OUT: track 0.00 -> 44.5 mm
- net /A_MSS_IN: track 0.00 -> 36.8 mm, vias 0 -> 2
- net Net-(J1-Pad2): track 0.00 -> 34.7 mm
- net Net-(J3-Pad3): track 32.4 -> 0.00 mm
- net GND: track 71.5 -> 103.3 mm, vias 26 -> 51
- net /S_MSS_IN: track 0.00 -> 30.9 mm, vias 0 -> 2
- net /MSS_OCC: track 29.5 -> 0.00 mm, vias 3 -> 0
- net Net-(J2-Pad4): track 28.5 -> 0.00 mm, vias 4 -> 0
- net Net-(J3-Pad8): track 28.1 -> 0.00 mm, vias 1 -> 0
- net Net-(J4-Pad3): track 0.00 -> 28.0 mm
- net Net-(J3-Pad7): track 27.4 -> 0.00 mm, vias 1 -> 0
- net Net-(J2-Pad1): track 27.4 -> 0.00 mm, vias 2 -> 0
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- added copper zone on F.Cu, net +5V
- removed copper zone on B.Cu, net /MSS_GND
- removed copper zone on F.Cu, net /~{CAL_SW}
Other:
- board size 73.7 x 38.1 mm -> 69.8 x 63.5 mm
- board text added: "ADV APRCH"
- board text added: "APRCH"
- board text added: "ATLAS J1->"
- board text added: "ATLAS J2->"
- board text added: "Atlas->MSS"
- board text added: "CURR BLOCK"
- board text added: "Iowa Scaled Engineering MSS-ATLASADAPTER v1.0 www.iascaled.com ©2024"
- board text added: "MSS <-"
- board text added: "MSS->Atlas"
- board text added: "POWER ON"
- board text added: "STATUS LIGHTS"
- board text removed: "CAL"
- board text removed: "DETECT"
- board text removed: "Iowa Scaled Engineering MSS-CROSSOVER v2.0 www.iascaled.com ©2024"
- board text removed: "MSS"
- board text removed: "PWR"
